File: kicad/nixie_clock/nixie_clock.kicad_sch (KiCad schematic)
At the start: 227 parts, among them Q1 STD10N60M2, U1 TPS40210DGQR, U2 STM32G0B1CBT6, U3 AP63203QWU-7, U4 TCAN334GDR, U5 SN74HC595DR, U6 SN74HC595DR, U7 SN74HC595DR, U8 SN75468DR, U9 SN75468DR, Y1 8MHz

Commit message: KiCad回路図に標準シンボル定義を埋め込む
Parts:
- D1: symbol Device:D_Fast -> Device:D
- QAH1, QAH2, QAH3, QAH4, QAH5, QAH6: symbol Transistor_BJT:MMBTA92 -> Transistor_BJT:Q_PNP_BEC
- QAL1, QAL2, QAL3, QAL4, QAL5, QAL6, QCOL1, QCOL2, QCOL3, QCOL4: symbol Transistor_BJT:MMBTA42 -> Transistor_BJT:Q_NPN_BEC
- U2: symbol MCU_ST_STM32G0:STM32G0B1CBTx -> MCU_ST_STM32G0:STM32G0B1C_B-C-E_Tx
- U3: symbol Regulator_Switching:AP63203WU -> Regulator_Switching:AP63200WU
- U4: symbol Interface_CAN_LIN:TCAN334G -> Interface_CAN_LIN:TCAN334

Commit message: KiCadフットプリントを確定して監査を追加
Parts:
- JCAN1: footprint TerminalBlock:TerminalBlock_Xinya_XY308-2.54-3P_1x03_P2.54mm_Horizontal -> nixie_clock_bom:OnShore_OSTVN03A150_1x03_P2.54mm_Horizontal
- JSWD1: footprint Connector_PinHeader_1.27mm:PinHeader_2x05_P1.27mm_Vertical_SMD -> nixie_clock_bom:Samtec_FTSH_105_01_F_DV_K_2x05_P1.27mm_Vertical_SMD
Changed lines of the file:
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@@
 			(effects (font (size 1.27 1.27)))
 		)
-		(property "Footprint" "TerminalBlock:TerminalBlock_Xinya_XY308-2.54-3P_1x03_P2.54mm_Horizontal"
+		(property "Footprint" "nixie_clock_bom:OnShore_OSTVN03A150_1x03_P2.54mm_Horizontal"
 			(at 254.00 330.20 0)
 			(hide yes)
@@
 			(effects (font (size 1.27 1.27)))
 		)
-		(property "Footprint" "Connector_PinHeader_1.27mm:PinHeader_2x05_P1.27mm_Vertical_SMD"
+		(property "Footprint" "nixie_clock_bom:Samtec_FTSH_105_01_F_DV_K_2x05_P1.27mm_Vertical_SMD"
 			(at 330.20 330.20 0)
 			(hide yes)

Commit message: KiCad回路図を機能ブロックで整理
Other:
- note added: "12V input, 170V boost controller and feedback parts"
- note added: "3.3V regulator, inductor, bulk/HF capacitors, enable bias"
- note added: "CAN transceiver, ESD protection, connector and termination"
- note added: "STM32, crystal, SWD connector, reset and logic support"
- note added: "Shift registers, sink drivers, anode switches, current/bias resistors"
- note added: "Six IN-12 sockets, 12 receptacle pins per tube"
- note added: "制御系 / CAN Interface"
- note added: "制御系 / MCU, Clock, Debug"
- note added: "表示管ソケット / IN-12"
- note added: "表示駆動系 / Nixie Drivers"
- note added: "電源系 / 3.3V Buck"
- note added: "電源系 / HV Boost"
- moved on the sheet: C3V3HF1, C3V3IN1, C3V3IN2, C3V3OUT1, C3V3OUT2, CBOOT1, CBP1, CCOMP1, CDEC1, CDEC2, CDEC3, CDEC4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

Commit message: 電源回路図をワイヤ配線で整理
Connections:
- net +12V_IN: now reaches C3V3HF1.1
- net +12V_IN: now also C3V3IN1.1, C3V3IN2.1, FHV1.1, R3V3EN1.1, U3.3 (IN)
- net GND: now reaches C3V3HF1.2
- net GND: now also C3V3IN1.2, C3V3IN2.2, C3V3OUT1.2, C3V3OUT2.2, CBP1.1, CBP1.2, CIFLT1.1, CIFLT1.2, CIN1.2, CIN2.2, CINB1.2, CINB2.2, COUT1.2, COUT2.2, COUT3.2, CRC1.2, CSS1.1, CSS1.2, CVDD1.2, Q1.3 (S), RBLD3.2, RENPD1.2, RFB6.2, RIFLT1.1, RIFLT1.2, RSNS1.1, RSNS1.2, U1.2 (SS), U1.6 (GND), U1.7 (ISNS), U1.9 (BP), U3.4 (GND)
- net HV170: now reaches COUT3.1
- net HV170: now also COUT1.1, COUT2.1, D1.1 (K), RBLD1.1, RFB1.1
- net at R3V3EN1.2: now also U3.2 (EN)
- net +3V3: now reaches U3.1 (FB)
- net +3V3: now also C3V3OUT1.1, C3V3OUT2.1, L2.2
- net at U3.5 (SW): now also CBOOT1.2, L2.1
- net at U3.6 (BST): now also CBOOT1.1
- net +12V_HV: now reaches CINB1.1
- net +12V_HV: now also CIN1.1, CIN2.1, CINB2.1, CVDD1.1, FHV1.2, L1.1, RRC1.1, U1.10 (VDD)
- net at RENPD1.1: now also REN1.2, U1.3 (DIS/EN)
- net at RFB1.2: now also RFB2.1
- net at RG1.1: now also U1.8 (GDRV)
- net at RG1.2: now also Q1.1 (G)
- net at RFB2.2: now also RFB3.1
- net at RBLD1.2: now also RBLD2.1
- net HV_DISABLE: now reaches REN1.1
- net at U1.1 (RC): now also CRC1.1, RRC1.2
- net at U1.4 (COMP): now also CCOMP1.1, CCOMP1.2, CHF1.1, CHF1.2, RCOMP1.1, RCOMP1.2, RFB5.2, RFB6.1, U1.5 (FB)
- net SW_HV: now reaches L1.2
- net SW_HV: now also D1.2 (A), Q1.2 (D), Q1.4 (D)
- net at RFB5.1: now also RFB4.2
- net at RBLD3.1: now also RBLD2.2
- net at RFB3.2: now also RFB4.1
Other:
- moved on the sheet: C3V3HF1, C3V3IN1, C3V3IN2, C3V3OUT1, C3V3OUT2, CBOOT1, CBP1, CCOMP1, CHF1, CIFLT1, CIN1, CIN2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
